File: board/billy/billy.kicad_sch (KiCad schematic)
At the start: 82 parts, among them J1 Screw_Terminal_01x02, J10 Screw_Terminal_01x02, J11 Screw_Terminal_01x03, J12 USB_B_Micro, J2 Conn_01x06, J3 Screw_Terminal_01x02, J4 Screw_Terminal_01x02, J5 Conn_01x02, J6 Conn_01x03, J7 Screw_Terminal_01x02, J8 Screw_Terminal_01x02, J9 Screw_Terminal_01x02, Q1 AOSS21311C, Q2 AOSS32334C, Q3 AOSS32334C, Q4 AOSS32334C, SW1 TS-1088-AR02016, U1 ESP32-S3-WROOM-1, U2 DRV8833PWPR, U3 MAX98357A, U4 DRV8833PWPR, U6 AP63203WU, U7 USBLC6-2SC6, U8 LM74700-Q1, U9 LM74700-Q1

Commit message: Replace USB-leg ideal diode with a passive Schottky and drop its now-redundant bypass cap
Parts:
- removed C21, C27: 100n, Capacitor_SMD:C_0603_1608Metric, symbol Device:C
- removed Q3: AOSS32334C, Package_TO_SOT_SMD:SOT-23, symbol Transistor_FET:AO3400A
- removed U9: LM74700-Q1, Package_TO_SOT_SMD:SOT-23-6, symbol Power_Management:LM74700
- added D2: B5817W, Diode_SMD:D_SOD-123, symbol Device:D
Connections:
- net BUCK_IN: now also D2.1 (K)
- net Vusb: now also D2.2 (A)
Other:
- moved on the sheet: C18, C20, C25, C26, D1, F1, F2, H1, H2, H3, H4, J11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

Commit message: Switch battery-leg RP MOSFET from AOSS21311C to the more common AO3401A
Parts:
- Q1: value AOSS21311C -> AO3401A; DigiKey Part 785-AOSS21311CCT-ND -> 785-1001-1-ND; LCSC Part C3280149 -> C15127; MP AOSS21311C -> AO3401A
Changed lines of the file:
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@@
 			)
 		)
-		(property "Value" "AOSS21311C"
+		(property "Value" "AO3401A"
 			(at 95.25 210.82 90)
 			(show_name no)
@@
 			)
 		)
-		(property "Datasheet" "https://www.aosmd.com/sites/default/files/res/datasheets/AOSS21311C.pdf"
+		(property "Datasheet" "https://www.aosmd.com/res/datasheets/AO3401A.pdf"
 			(at 91.44 212.09 0)
 			(hide yes)
@@
 			)
 		)
-		(property "Description" "Passive reverse-battery protection (self-biased, S=Vbatt/D=Vdrive/G=R19 pulldown); 30V Vds, 4.3A Id, P-Channel MOSFET, SOT-23"
+		(property "Description" "Passive reverse-battery protection (self-biased, S=Vbatt/D=Vdrive/G=R19 pulldown); 30V Vds, 4.0A Id, P-Channel MOSFET, SOT-23"
 			(at 95.25 217.17 0)
 			(hide yes)
@@
 			)
 		)
-		(property "LCSC Part" "C3280149"
+		(property "LCSC Part" "C15127"
 			(at 95.25 217.17 90)
 			(hide yes)
@@
 			)
 		)
-		(property "MP" "AOSS21311C"
+		(property "MP" "AO3401A"
 			(at 95.25 217.17 90)
 			(hide yes)
@@
 			)
 		)
-		(property "DigiKey Part" "785-AOSS21311CCT-ND"
+		(property "DigiKey Part" "785-1001-1-ND"
 			(at 95.25 217.17 90)
 			(hide yes)

Commit message: Replace repurposed MOTOR_RAIL->BUCK_IN leg's LM74700-Q1 with LTC4412 + AO3401A
Parts:
- removed C20: 100n, Capacitor_SMD:C_0603_1608Metric, symbol Device:C
- removed Q2: AOSS32334C, Package_TO_SOT_SMD:SOT-23, symbol Transistor_FET:AO3400A
- removed U8: LM74700-Q1, Package_TO_SOT_SMD:SOT-23-6, symbol Power_Management:LM74700
- added Q2: AO3401A, Package_TO_SOT_SMD:SOT-23, symbol Transistor_FET:AO3401A
- added U5: LTC4412, Package_TO_SOT_SMD:TSOT-23-6, symbol Power_Management:LTC4412xS6
- D2: Mouser Part (none) -> 833-B5817W-TP
Connections:
- net BUCK_IN: now also Q2.2 (S), U5.6 (SENSE)
- net GND: now also U5.2 (GND)
- net Vdrive renamed Vmot
- net Vmot: now also Q2.3 (D), U5.1 (VIN)
- new net: Q2.1 (G), U5.5 (GATE)
- no-connect marks 17 -> 19

Commit message: Switch status-LED gate FET (Q4) from AOSS32334C to the more common AO3400A
Parts:
- Q4: value AOSS32334C -> AO3400A; DigiKey Part 785-AOSS32334CCT-ND -> 785-1000-1-ND; LCSC Part C3280157 -> C20917; MP AOSS32334C -> AO3400A
Changed lines of the file:
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@@
 			)
 		)
-		(property "Value" "AOSS32334C"
+		(property "Value" "AO3400A"
 			(at 158.75 161.2899 0)
 			(show_name no)
@@
 			)
 		)
-		(property "Datasheet" "https://www.aosmd.com/res/datasheets/AOSS32334C.pdf"
+		(property "Datasheet" "https://www.aosmd.com/res/datasheets/AO3400A.pdf"
 			(at 157.48 163.83 0)
 			(hide yes)
@@
 			)
 		)
-		(property "Description" "30V Vds, 6.2A Id, N-Channel MOSFET, SOT-23"
+		(property "Description" "WS2812 VDD-gate low-side switch (D1 VSS return, gated by GPIO18/BOARD_STATUS_LED_EN); 30V Vds, 5.7A Id, N-Channel MOSFET, SOT-23"
 			(at 152.4 160.02 0)
 			(hide yes)
@@
 			)
 		)
-		(property "LCSC Part" "C3280157"
+		(property "LCSC Part" "C20917"
 			(at 152.4 160.02 0)
 			(hide yes)
@@
 			)
 		)
-		(property "MP" "AOSS32334C"
+		(property "MP" "AO3400A"
 			(at 152.4 160.02 0)
 			(hide yes)
@@
 			)
 		)
-		(property "DigiKey Part" "785-AOSS32334CCT-ND"
+		(property "DigiKey Part" "785-1000-1-ND"
 			(at 152.4 160.02 0)
 			(hide yes)

Commit message: Gate the photocell divider off BOARD_AWAKE_EN, shared with the status LED's supply gate
Parts:
- added Q6: AO3400A, Package_TO_SOT_SMD:SOT-23, symbol Transistor_FET:AO3400A
Connections:
- net GND: now also Q6.2 (S); no longer R5.2
- net GPIO18: now also Q6.1 (G)
- new net: Q6.3 (D), R5.2
Other:
- moved on the sheet: J1, J2, R5, TP5, TP6

Commit message: Gate Vmotor-sense divider off BOARD_PERIPHERALS_EN (Q7) and merge sensors/status_led into peripherals.c
Parts:
- added Q7: AO3400A, Package_TO_SOT_SMD:SOT-23, symbol Transistor_FET:AO3400A
Connections:
- net GND: now also Q7.2 (S); no longer R15.2
- net GPIO18: now also Q7.1 (G)
- new net: Q7.3 (D), R15.2
Other:
- moved on the sheet: C18, D1, J1, Q4, Q6, R17, R18, R5

Commit message: Replace fuse holders with SMD fuses to save cost
Parts:
- C12, C5: DigiKey Part 1276-1028-1-ND -> 1276-1009-1-ND; MP CL05B103KB5NNNC -> CL10B103KB8NNNC
- F1, F2: footprint Fuse:Fuseholder_Littelfuse_Nano2_154x -> Fuse:Fuse_Littelfuse-NANO2-451_453; DigiKey Part F1310CT-ND -> F3147CT-ND; MP 0154005.DRT -> 0454005.MR; Mouser Part 576-0154005.DRT -> 576-0454005.MR
Changed lines of the file:
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@@
 			)
 		)
-		(property "Description" "Gate pulldown for Q1 (AOSS21311C) self-biased P-FET battery reverse-polarity protection"
+		(property "Description" "Resistor"
 			(at 95.25 227.33 0)
 			(hide yes)
@@
 			)
 		)
-		(property "Footprint" "Fuse:Fuseholder_Littelfuse_Nano2_154x"
+		(property "Footprint" "Fuse:Fuse_Littelfuse-NANO2-451_453"
 			(at 62.23 216.408 90)
 			(hide yes)
@@
 			)
 		)
-		(property "MP" "0154005.DRT"
+		(property "MP" "0454005.MR"
 			(at 62.23 214.63 90)
 			(hide yes)
@@
 			)
 		)
-		(property "DigiKey Part" "F1310CT-ND"
+		(property "DigiKey Part" "F3147CT-ND"
 			(at 62.23 214.63 90)
 			(hide yes)
@@
 			)
 		)
-		(property "Mouser Part" "576-0154005.DRT"
+		(property "Mouser Part" "576-0454005.MR"
 			(at 62.23 214.63 90)
 			(hide yes)
@@
 			)
 		)
-		(property "Description" "Unpolarized capacitor, 16V, X7R"
+		(property "Description" "Unpolarized capacitor"
 			(at 201.93 96.52 0)
 			(hide yes)
@@
 			)
 		)
-		(property "MP" "CL05B103KB5NNNC"
+		(property "MP" "CL10B103KB8NNNC"
 			(at 201.93 96.52 0)
 			(hide yes)
@@
 			)
 		)
-		(property "DigiKey Part" "1276-1028-1-ND"
+		(property "DigiKey Part" "1276-1009-1-ND"
 			(at 201.93 96.52 0)
 			(hide yes)
@@
 			)
 		)
-		(property "MP" "CL05B103KB5NNNC"
+		(property "MP" "CL10B103KB8NNNC"
 			(at 201.93 143.51 0)
 			(hide yes)
@@
 			)
 		)
-		(property "DigiKey Part" "1276-1028-1-ND"
+		(property "DigiKey Part" "1276-1009-1-ND"
 			(at 201.93 143.51 0)
 			(hide yes)
@@
 			)
 		)
-		(property "Footprint" "Fuse:Fuseholder_Littelfuse_Nano2_154x"
+		(property "Footprint" "Fuse:Fuse_Littelfuse-NANO2-451_453"
 			(at 62.23 246.888 90)
 			(hide yes)
@@
 			)
 		)
-		(property "MP" "0154005.DRT"
+		(property "MP" "0454005.MR"
 			(at 62.23 245.11 90)
 			(hide yes)
@@
 			)
 		)
-		(property "DigiKey Part" "F1310CT-ND"
+		(property "DigiKey Part" "F3147CT-ND"
 			(at 62.23 245.11 90)
 			(hide yes)
@@
 			)
 		)
-		(property "Mouser Part" "576-0154005.DRT"
+		(property "Mouser Part" "576-0454005.MR"
 			(at 62.23 245.11 90)
 			(hide yes)
@@
 			)
 		)
-		(property "Description" "Resistor -- Vmotor-sense divider top leg (see R15, bottom leg); Vdrive to R13 to GPIO8/ADC node"
+		(property "Description" "Resistor"
 			(at 154.94 82.55 0)
 			(hide yes)
@@
 			)
 		)
-		(property "Description" "Resistor -- Vmotor-sense divider bottom leg (see R13, top leg)"
+		(property "Description" "Resistor"
 			(at 154.94 92.71 0)
 			(hide yes)

Commit message: Replace motor screw terminals with 1x6 block to save space and part count
Parts:
- removed J7, J8, J9: Screw_Terminal_01x02, TerminalBlock:TerminalBlock_Xinya_XY308-2.54-2P_1x02_P2.54mm_Horizontal, symbol Connector:Screw_Terminal_01x02
- added J7: Screw_Terminal_01x06, TerminalBlock:TerminalBlock_Xinya_XY308-2.54-6P_1x06_P2.54mm_Horizontal, symbol Connector:Screw_Terminal_01x06
Connections:
- net at U4.2 (AOUT1): now also J7.5 (Pin_5)
- net at U4.4 (AOUT2): now also J7.6 (Pin_6)
- net at U2.2 (AOUT1): now also J7.1 (Pin_1)
- net at U2.4 (AOUT2): now also J7.2 (Pin_2)
- net at U2.5 (BOUT2): now also J7.4 (Pin_4)
- net at U2.7 (BOUT1): now also J7.3 (Pin_3)
